File: D24cpu.kicad_sch (KiCad schematic)
At the start: 20 parts, among them J2 NEM651, J4 Conn_01x01, J5 Conn_01x01, J6 Conn_01x01, J7 WS28xx data, J8 WS28xx GND, J9 WS28xx power, U1 AVR-64DA32

Commit message: refined BOM
Parts:
- D1: value LED pink -> LED; LCSC Part # (none) -> C130724
Changed lines of the file:
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@@
 			)
 		)
-		(property "Value" "LED pink"
+		(property "Value" "LED"
 			(at 207.01 73.152 0)
 			(show_name no)
@@
 			)
 		)
-		(property "Description" ""
+		(property "Description" "-30℃~+85℃ 130° 2.6V~3.6V 20mA 45mcd 463nm~475nm 465nm 72mW Blue Discrete Diode 0402 LED Indication - Discrete ROHS"
 			(at 207.01 67.31 0)
-			(show_name no)
-			(do_not_autoplace no)
-			(effects
-				(font
-					(size 1.27 1.27)
-				)
-			)
-		)
-		(property "LCSC Part #" ""
+			(hide yes)
+			(show_name no)
+			(do_not_autoplace no)
+			(effects
+				(font
+					(size 1.27 1.27)
+				)
+			)
+		)
+		(property "LCSC Part #" "C130724"
 			(at 207.01 67.31 0)
 			(hide yes)
@@
 			)
 		)
-		(property "Description" "Schottky diode, small symbol"
+		(property "Description" "1 Independent 150uA@40V 2A 40V 550mV@2A 0603 Schottky Diodes ROHS"
 			(at 54.61 129.54 0)
 			(hide yes)
